Commit message: Lower joint effort limits to reduce effects of bad control impulses.

File: ow_lander/urdf/lander.xacro (robot description, xacro)
@@ -158,5 +158,5 @@
       xyz="0 0 -1" />
     <dynamics damping="50.0" />
-    <limit effort="1000.0" velocity="0.15" lower="-1.8" upper="1.8"/>
+    <limit effort="100.0" velocity="0.15" lower="-1.8" upper="1.8"/>
   </joint>
   <transmission name="shou_yaw_transmission">
@@ -234,5 +234,5 @@
       xyz="0 0 -1" />
     <dynamics damping="50.0" />
-    <limit effort="1000.0" velocity="0.2" lower="0.05" upper="2.2"/>
+    <limit effort="100.0" velocity="0.2" lower="0.05" upper="2.2"/>
   </joint>
   <transmission name="shou_pitch_transmission">
@@ -310,5 +310,5 @@
       xyz="0 0 -1" />
     <dynamics damping="50.0" />
-    <limit effort="1000.0" velocity="0.2" />
+    <limit effort="60.0" velocity="0.2" />
   </joint>
   <transmission name="prox_pitch_transmission">
@@ -386,5 +386,5 @@
       xyz="0 0 1" />
     <dynamics damping="50.0" />
-    <limit effort="1000.0" velocity="0.2" />
+    <limit effort="20.0" velocity="0.2" />
   </joint>
   <transmission name="dist_pitch_transmission">
@@ -471,5 +471,5 @@
       xyz="0 0 -1" />
     <dynamics damping="50.0" />
-    <limit effort="1000.0" velocity="0.2" />
+    <limit effort="10.0" velocity="0.2" />
   </joint>
   <transmission name="hand_yaw_transmission">
@@ -573,5 +573,5 @@
       xyz="0 0 -1" />
     <dynamics damping="50" />
-    <limit effort="1000.0" velocity="0.4" />
+    <limit effort="10.0" velocity="0.4" />
   </joint>
   <transmission name="scoop_yaw_transmission">
@@ -718,5 +718,5 @@
       xyz="0 0 -1" />
     <dynamics damping="50" />
-    <limit effort="1000.0" velocity="0.4" />
+    <limit effort="40.0" velocity="0.4" />
   </joint>
   <transmission name="ant_pan_transmission">
@@ -794,5 +794,5 @@
       xyz="0 0 -1" />
     <dynamics damping="50" />
-    <limit effort="1000.0" velocity="0.4" />
+    <limit effort="40.0" velocity="0.4" />
   </joint>
   <transmission name="ant_tilt_transmission">
